File: board/DC26Badge.kicad_pcb (KiCad board)
At the start: 2 copper layers, 6 parts, among them U1 HT16K33-28

Commit message: Rearrange, create skeleton firmware.
Connections:
- U1 pad 22: /N -> /M
- U1 pad 23: /M -> /N
Routing:
- net /M: track 88.1 -> 104.0 mm, vias 3 -> 4
- net /N: track 85.4 -> 100.9 mm, vias 3 -> 4
- net /L: track 109.0 -> 109.7 mm
- net /DP: track 95.4 -> 96.1 mm
Changed lines of the file:
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@@
     (thickness 1.6)
     (drawings 0)
-    (tracks 340)
+    (tracks 354)
     (zones 0)
     (modules 6)
@@
       (net 24 /DIG3))
     (pad 23 smd rect (at -1.905 4.25) (size 0.76 1.2) (layers B.Cu B.Paste B.Mask)
-      (net 13 /M))
+      (net 11 /N))
     (pad 6 smd rect (at -1.905 -4.25) (size 0.76 1.2) (layers B.Cu B.Paste B.Mask)
       (net 27 /DIG4))
     (pad 22 smd rect (at -0.635 4.25) (size 0.76 1.2) (layers B.Cu B.Paste B.Mask)
-      (net 11 /N))
+      (net 13 /M))
     (pad 7 smd rect (at -0.635 -4.25) (size 0.76 1.2) (layers B.Cu B.Paste B.Mask)
       (net 29 /DIG5))
@@
   (segment (start 117.57 46.5) (end 117.57 45.25) (width 0.25) (layer B.Cu) (net 4))
   (segment (start 117.57 45.25) (end 118.07 44.75) (width 0.25) (layer B.Cu) (net 4))
-  (segment (start 146.5636 59.85501) (end 159.51001 59.85501) (width 0.25) (layer B.Cu) (net 5))
-  (segment (start 159.51001 59.85501) (end 161.03 61.375) (width 0.25) (layer B.Cu) (net 5))
-  (segment (start 161.03 61.375) (end 161.03 61.74) (width 0.25) (layer B.Cu) (net 5))
+  (segment (start 161.03 61.375) (end 159.51001 59.85501) (width 0.25) (layer B.Cu) (net 5))
+  (segment (start 161.03 61.74) (end 161.03 61.375) (width 0.25) (layer B.Cu) (net 5))
+  (segment (start 159.51001 59.85501) (end 145.85501 59.85501) (width 0.25) (layer B.Cu) (net 5))
+  (segment (start 145.85501 59.85501) (end 145.175 59.175) (width 0.25) (layer B.Cu) (net 5))
+  (segment (start 145.175 59.175) (end 145.175 58.25) (width 0.25) (layer B.Cu) (net 5))
   (segment (start 145.175 58.25) (end 145.175 58.46641) (width 0.25) (layer B.Cu) (net 5))
-  (segment (start 145.175 58.46641) (end 146.5636 59.85501) (width 0.25) (layer B.Cu) (net 5))
   (segment (start 184 64.25) (end 184 61.77) (width 0.25) (layer F.Cu) (net 5))
   (segment (start 184 61.77) (end 184.03 61.74) (width 0.25) (layer F.Cu) (net 5))
@@
   (segment (start 109.95 46.5) (end 109.95 46.135) (width 0.25) (layer B.Cu) (net 10))
   (via (at 179 43.25) (size 0.8) (drill 0.4) (layers F.Cu B.Cu) (net 10))
+  (segment (start 133.25 56.25) (end 130.41 59.09) (width 0.25) (layer F.Cu) (net 11))
+  (segment (start 140 56.25) (end 133.25 56.25) (width 0.25) (layer F.Cu) (net 11))
+  (segment (start 130.41 59.09) (end 130.41 61.74) (width 0.25) (layer F.Cu) (net 11))
+  (segment (start 140.095 56.345) (end 140 56.25) (width 0.25) (layer B.Cu) (net 11))
+  (segment (start 140.095 58.25) (end 140.095 56.345) (width 0.25) (layer B.Cu) (net 11))
+  (via (at 140 56.25) (size 0.8) (drill 0.4) (layers F.Cu B.Cu) (net 11))
   (segment (start 130.5 66.5) (end 153.5 66.5) (width 0.25) (layer B.Cu) (net 11))
   (segment (start 112.987341 66.5) (end 130.5 66.5) (width 0.25) (layer B.Cu) (net 11))
@@
   (segment (start 107.41 46.5) (end 107.41 46.135) (width 0.25) (layer B.Cu) (net 12))
   (segment (start 107.41 46.135) (end 111.045 42.5) (width 0.25) (layer B.Cu) (net 12))
+  (segment (start 141.5 56.25) (end 141.5 58.115) (width 0.25) (layer B.Cu) (net 13))
+  (segment (start 141.5 58.115) (end 141.365 58.25) (width 0.25) (layer B.Cu) (net 13))
+  (segment (start 149.25 56.25) (end 141.5 56.25) (width 0.25) (layer F.Cu) (net 13))
+  (segment (start 150.87 57.87) (end 149.25 56.25) (width 0.25) (layer F.Cu) (net 13))
+  (via (at 141.5 56.25) (size 0.8) (drill 0.4) (layers F.Cu B.Cu) (net 13))
+  (segment (start 150.87 61.74) (end 150.87 57.87) (width 0.25) (layer F.Cu) (net 13))
   (segment (start 127.75 67.25) (end 150.75 67.25) (width 0.25) (layer B.Cu) (net 13))
   (segment (start 111.197341 67.25) (end 127.75 67.25) (width 0.25) (layer B.Cu) (net 13))
@@
   (segment (start 144.285 52.25) (end 171.25 52.25) (width 0.25) (layer B.Cu) (net 16))
   (via (at 171.25 52.25) (size 0.8) (drill 0.4) (layers F.Cu B.Cu) (net 16))
-  (segment (start 138.825 58.46641) (end 137.29141 60) (width 0.25) (layer B.Cu) (net 17))
+  (segment (start 122.79 60.46) (end 123.25 60) (width 0.25) (layer B.Cu) (net 17))
+  (segment (start 123.25 60) (end 138.25 60) (width 0.25) (layer B.Cu) (net 17))
+  (segment (start 122.79 61.74) (end 122.79 60.46) (width 0.25) (layer B.Cu) (net 17))
+  (segment (start 138.25 60) (end 138.825 59.425) (width 0.25) (layer B.Cu) (net 17))
+  (segment (start 138.825 59.425) (end 138.825 58.25) (width 0.25) (layer B.Cu) (net 17))
   (segment (start 138.825 58.25) (end 138.825 58.46641) (width 0.25) (layer B.Cu) (net 17))
-  (segment (start 137.29141 60) (end 123.25 60) (width 0.25) (layer B.Cu) (net 17))
-  (segment (start 123.25 60) (end 122.79 60.46) (width 0.25) (layer B.Cu) (net 17))
-  (segment (start 122.79 60.46) (end 122.79 61.74) (width 0.25) (layer B.Cu) (net 17))
   (segment (start 122.75 68) (end 145.75 68) (width 0.25) (layer B.Cu) (net 17))
   (segment (start 106.867341 68) (end 122.75 68) (width 0.25) (layer B.Cu) (net 17))

Commit message: First pass of prototype PCB layout.
Parts:
- added C2: 4.7u, Capacitor_SMD:C_0603_1608Metric, F.Cu at (154.9, 33.8)
- added C3: 0.1u, Capacitor_SMD:C_0603_1608Metric, F.Cu at (154.9, 31.6)
- added C4: 0.1u, Capacitor_SMD:C_0603_1608Metric, F.Cu at (112.8, 26.0)
- added C5: 0.1u, Capacitor_SMD:C_0603_1608Metric, F.Cu at (133.1, 32.4)
- added D1: LED, LED_SMD:LED_0603_1608Metric, F.Cu at (126.8, 24.7)
- added J1: PWR_HDR, PinHeaders:Pin_Header_Straight_1x02_Pitch2.54mm, F.Cu at (173.6, 35.3)
- added J2: PWR_CONN, Connector_JST:JST_PH_S2B-PH-SM4-TB_1x02_P2.00mm_Horizontal, F.Cu at (182.6, 33.9)
- added J3: VOLTMETER, PinHeaders:Pin_Header_Straight_1x02_Pitch2.54mm, F.Cu at (168.8, 35.3)
- added J4: AMMETER, PinHeaders:Pin_Header_Straight_1x02_Pitch2.54mm, F.Cu at (163.8, 31.1)
- added J5: Cortex_SWD, Connector_PinHeader_1.27mm:PinHeader_2x05_P1.27mm_Vertical_SMD, F.Cu at (116.7, 31.9)
- added R1: 0.1, DC26badge:FC4T, F.Cu at (162.5, 35.8)
- added R2: 1k, Resistor_SMD:R_0603_1608Metric, F.Cu at (123.1, 24.7)
- added R3: 1k, Resistor_SMD:R_0603_1608Metric, F.Cu at (121.8, 32.2)
- added SW1: JOYSTICK, DC26badge:JOYSTICK, F.Cu at (142.2, 32.6)
- added SW2: SW_Push, Button_Switch_SMD:SW_SPST_SKQG, F.Cu at (127.9, 32.3)
- added TP1: PWRTP, TestPoint:TestPoint_2Pads_Pitch2.54mm_Drill0.8mm, F.Cu at (153.7, 36.5)
- added U2: BT832, DC26badge:BT832, F.Cu at (105.0, 33.2)
Routing:
- net /DN: track 0.00 -> 47.9 mm, vias 0 -> 2
- net /RESET: track 0.00 -> 47.3 mm, vias 0 -> 2
- net /RT: track 0.00 -> 46.2 mm, vias 0 -> 2
- net /UP: track 0.00 -> 41.7 mm, vias 0 -> 2
- net /CTR: track 0.00 -> 40.1 mm, vias 0 -> 2
- net /LT: track 0.00 -> 38.0 mm, vias 0 -> 2
- net VDD: track 49.7 -> 25.0 mm, vias 0 -> 1
- net /SWDCLK: track 0.00 -> 22.9 mm
- net /SWDIO: track 0.00 -> 22.6 mm
- net /LED1: track 0.00 -> 21.0 mm, vias 0 -> 2
- net /P_IN: track 0.00 -> 16.4 mm
- net GND: track 46.9 -> 39.5 mm, vias 0 -> 6
- net Net-(J4-Pad2): track 0.00 -> 4.11 mm
- net Net-(J4-Pad1): track 0.00 -> 4.08 mm
- net Net-(D1-Pad1): track 0.00 -> 1.95 mm
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- added copper zone on B.Cu, net GND
- added copper zone on F.Cu, net VDD
Other:
- board outline added: 94 x 48 mm
