File: board/_autosave-DC26Badge.kicad_pcb (KiCad board)
At the start: 2 copper layers, 94 x 46.5 mm, 23 parts, among them J1 PWR_HDR, J2 PWR_CONN, J3 VOLTMETER, J4 AMMETER, J5 Cortex_SWD, SW1 JOYSTICK, SW2 SW_Push, U1 HT16K33-28, U2 BT832

Commit message: Prototype R1.
Parts:
- renumbered SW2 to RESET, J5 to SWD
Changed lines of the file:
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@@
     (tags "SPST Button Switch")
     (attr smd)
-    (fp_text reference SW2 (at 0 -3.6 180) (layer F.SilkS)
+    (fp_text reference RESET (at 0 -3.6 180) (layer F.SilkS)
       (effects (font (size 1 1) (thickness 0.15)))
     )
@@
     (tags "Surface mounted pin header SMD 2x05 1.27mm double row")
     (attr smd)
-    (fp_text reference J5 (at 0 -4.235) (layer F.SilkS)
-      (effects (font (size 1 1) (thickness 0.15)))
-    )
+    (fp_text reference SWD (at 0 -4.235) (layer F.SilkS)
+      (effects (font (size 1 1) (thickness 0.15)))
+    )
